File: LARS.sch (EAGLE design)
At the start: 11 parts, among them IC1 L293D, IC2 L293D, IC3 L293D, IC4 L293D, IC5 L293D, U1 ARDUINO-MEGAFULL

Commit message: placa dia 12/09
Parts:
- removed D1: SFH482, led:SFH482
- removed IC1, IC2, IC3, IC4, IC5: L293D, st-microelectronics:L293D
- added JP10, JP11, JP12, JP5, JP6, JP7, JP8, JP9: (no value), pinhead:PINHD-1X2
- added JP13: (no value), pinhead:PINHD-1X3
- added LED1: TLLG4400, led:TLLG4400
- added MOTOR12, MOTOR34, STEP1, STEP2: L293D, st-microelectronics:L293D
Connections:
- removed net N$1: IC2.1-2EN, IC3.1-2EN
- removed net N$10: IC2.4A, IC3.4A
- removed net N$11: IC2.4Y, IC3.4Y
- removed net N$12: IC2.GND3, IC3.GND3
- removed net N$13: IC2.GND4, IC3.GND4
- removed net N$14: IC2.3Y, IC3.3Y
- removed net N$15: IC2.3A, IC3.3A
- removed net N$16: IC2.3-4EN, IC3.3-4EN
- removed net N$2: IC2.1A, IC3.1A
- removed net N$6: IC2.2Y, IC3.2Y
- removed net N$7: IC2.2A, IC3.2A
- removed net N$8: IC2.VCC2, IC3.VCC2
- removed net N$9: IC2.VCC1, IC3.VCC1
- new net GND: JP1.3, JP13.3, JP2.3, JP3.3, JP4.3, LED1.C, MOTOR12.GND1, MOTOR12.GND2, MOTOR12.GND3, MOTOR12.GND4, MOTOR34.GND1, MOTOR34.GND2, MOTOR34.GND3, MOTOR34.GND4, STEP1.GND1, STEP1.GND2, STEP1.GND3, STEP1.GND4, STEP2.GND1, STEP2.GND2, STEP2.GND3, STEP2.GND4, U1.GND@0, U1.GND@1, U1.GND@2, U1.GND@3, U1.GND@4
- new net INB1: MOTOR12.2A, U1.6
- new net INC1: MOTOR12.3A, U1.7
- new net INC2: STEP2.3A
- new net IND1: MOTOR12.4A, U1.8
- new net SERVO1: JP1.1, U1.13
- new net SERVO2: JP2.1, U1.12
- new net SERVO3: JP3.1, U1.11
- new net SERVO4: JP4.1, U1.10
- new net SERVO5: JP13.1, U1.9
- new net STP1: JP5.2, STEP1.1Y
- new net STP10: JP9.1, MOTOR12.2Y
- new net STP11: JP10.2, MOTOR12.3Y
- new net STP12: JP10.1, MOTOR12.4Y
- new net STP13: JP11.2, MOTOR34.1Y
- new net STP14: JP11.1, MOTOR34.2Y
- new net STP15: JP12.2, MOTOR34.3Y
- new net STP16: JP12.1, MOTOR34.4Y
- new net STP2: JP5.1, STEP1.2Y
- new net STP3: JP6.2, STEP1.3Y
- new net STP4: JP6.1, STEP1.4Y
- new net STP5: JP7.2, STEP2.1Y
- new net STP6: JP7.1, STEP2.2Y
- new net STP7: JP8.2, STEP2.3Y
- new net STP8: JP8.1, STEP2.4Y
- new net STP9: JP9.2, MOTOR12.1Y
- new net VCC: JP1.2, JP13.2, JP2.2, JP3.2, JP4.2, LED1.A, MOTOR12.1-2EN, MOTOR12.3-4EN, MOTOR12.VCC1, MOTOR34.1-2EN, MOTOR34.3-4EN, MOTOR34.VCC1, STEP1.1-2EN, STEP1.3-4EN, STEP1.VCC1, STEP2.1-2EN, STEP2.3-4EN, STEP2.VCC1, U1.5V@0, U1.5V@1, U1.5V@2
- new net VCC2: MOTOR12.VCC2, MOTOR34.VCC2, STEP1.VCC2, STEP2.VCC2
- net N$3: now also U1.5; no longer IC2.1Y, IC3.1Y
- net N$4: now also U1.4; no longer IC2.GND1, IC3.GND1
- net N$5: now also U1.3; no longer IC2.GND2, IC3.GND2
Other:
- moved on the sheet: JP1, JP2, JP3, JP4

Commit message: parei de mexer na placa pra tentar fazer o robô móvel
Parts:
- added JP14, JP15, JP16, JP17, JP19, JP20, JP21, JP22, JP23, JP24, JP25, JP26, JP27, JP28, JP30, JP31, JP32, JP33: (no value), pinhead:PINHD-1X1
- added JP18, JP29: (no value), pinhead:PINHD-1X2
- added JP34, JP35, JP36, JP37, JP38: (no value), pinhead:PINHD-1X3
Connections:
- removed net INC2: STEP2.3A
- removed net N$3: U1.5
- new net OUTB2: MOTOR34.2A, U1.26
- new net OUTD2: MOTOR34.4A, U1.5
- new net PIN2: JP21.1, JP22.1, MOTOR34.1A, U1.2
- new net PIN24: JP23.1, JP25.1, MOTOR34.3A, U1.24
- new net PIN38: JP19.1, JP20.1, MOTOR12.1A, U1.36
- new net STPA1: JP17.1, JP24.1, STEP1.1A, U1.52
- new net STPA2: JP26.1, JP31.1, STEP2.1A, U1.48
- new net STPB1: JP14.1, JP30.1, STEP1.2A, U1.50
- new net STPB2: STEP2.2A, U1.46
- new net STPC1: JP16.1, JP32.1, STEP1.3A, U1.40
- new net STPC2: STEP2.3A, U1.44
- new net STPD1: JP15.1, JP33.1, STEP1.4A, U1.38
- new net STPD2: JP27.1, JP28.1, STEP2.4A, U1.42
- new net VCC3: JP29.2, STEP1.VCC2, STEP2.VCC2
- net GND: now also JP18.1, JP29.1, JP34.3, JP35.3, JP36.3, JP37.3, JP38.3
- net SERVO1: now also JP35.1
- net SERVO2: now also JP34.1
- net SERVO3: now also JP36.1
- net SERVO4: now also JP37.1
- net SERVO5: now also JP38.1
- net STP1: now also STEP2.1Y; no longer STEP1.1Y
- net STP13: now also STEP1.1Y; no longer MOTOR34.1Y
- net STP14: now also STEP1.2Y; no longer MOTOR34.2Y
- net STP15: now also STEP1.3Y; no longer MOTOR34.3Y
- net STP16: now also STEP1.4Y; no longer MOTOR34.4Y
- net STP2: now also STEP2.2Y; no longer STEP1.2Y
- net STP3: now also STEP2.3Y; no longer STEP1.3Y
- net STP4: now also STEP2.4Y; no longer STEP1.4Y
- net STP5: now also MOTOR34.1Y; no longer STEP2.1Y
- net STP6: now also MOTOR34.2Y; no longer STEP2.2Y
- net STP7: now also MOTOR34.3Y; no longer STEP2.3Y
- net STP8: now also MOTOR34.4Y; no longer STEP2.4Y
- net VCC: now also JP34.2, JP35.2, JP36.2, JP37.2, JP38.2
- net VCC2: now also JP18.2; no longer STEP1.VCC2, STEP2.VCC2
Other:
- moved on the sheet: JP10, JP11, JP12, JP5, JP6, JP7, JP8, JP9, LED1, MOTOR12, MOTOR34, STEP1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
